Commit message: added gazebo sim

File: description/robot_core.xacro (robot description, xacro)
@@ -44,4 +44,9 @@
     </xacro:inertial_box>
 </link>
+<!--now we just add gazebo tags that tell gazebo to do certain things while simulation-->
+<!--first thing we can tackle is fixin up the colors, basically any link that has a visual tag, we need to add a gazebo tag to add the colors in gazebo during the simulation-->
+<gazebo reference="chassis">
+    <material>Gazebo/White</material>
+</gazebo>
 <!-- LEFT WHEEL LINK -->
 <joint name="left_wheel_joint" type="continuous">
@@ -67,4 +72,7 @@
     </xacro:inertial_cylinder>
 </link>
+<gazebo reference="left_wheel">
+    <material>Gazebo/Blue</material>
+</gazebo>
 <!--RIGHT WHEEL LINK-->
 <joint name="right_wheel_joint" type="continuous">
@@ -90,4 +98,7 @@
     </xacro:inertial_cylinder>
 </link>
+<gazebo reference="right_wheel">
+    <material>Gazebo/Blue</material>
+</gazebo>
 <!--CASTER WHEEL LINK-->
 <joint name="caster_wheel_joint" type="fixed">
@@ -112,4 +123,9 @@
     </xacro:inertial_sphere>
 </link>
+<gazebo reference="caster_wheel">
+    <material>Gazebo/Black</material>
+    <mu1 value="0.0001"/>
+    <mu2 value="0.0001"/>
+</gazebo>
 <!--STEPS TO RUN
 1. rebuilt the files : colcon build symlink-install in the dev_ws dir
